File: ESP32-breakout-SMD.kicad_pcb (KiCad board)
At the start: 2 copper layers, 35.1 x 50.4 mm, 16 parts, among them J1 Conn_01x14, J2 Conn_01x14, J3 Conn_01x02_Male, J4 Conn_01x04_Male, J5 Conn_01x04_Male, SW1 RESET, SW2 BOOT, U1 ESP32-WROOM

Commit message: fix: 微修正
Parts:
- removed the REF** at (165.5, 128.2)
- removed the REF** at (163.4, 128.2)
- added REF**: PinHeader_1x01_P2.54mm_Vertical, Connector_PinHeader_2.54mm:PinHeader_1x01_P2.54mm_Vertical, F.Cu at (166.2, 128.3)
- added REF**: PinHeader_1x01_P2.54mm_Vertical, Connector_PinHeader_2.54mm:PinHeader_1x01_P2.54mm_Vertical, F.Cu at (163.4, 128.2)
- C1, C2, C4: footprint Capacitor_SMD:C_0805_2012Metric -> Capacitor_SMD:C_0805_2012Metric_Pad1.15x1.40mm_HandSolder
- C3: footprint Capacitor_SMD:C_1206_3216Metric -> Capacitor_SMD:C_1206_3216Metric_Pad1.42x1.75mm_HandSolder
- R1: footprint Resistor_SMD:R_0805_2012Metric -> Resistor_SMD:R_0805_2012Metric_Pad1.15x1.40mm_HandSolder
- REF**: value PinHeader_1x01_P1.27mm_Vertical -> PinHeader_1x01_P2.54mm_Vertical; footprint Connector_PinHeader_1.27mm:PinHeader_1x01_P1.27mm_Vertical -> Connector_PinHeader_2.54mm:PinHeader_1x01_P2.54mm_Vertical
- moved REF** 0.81 mm to (160.6, 128.2)
- moved J3 0.20 mm to (151.1, 138.8)
- moved J4 0.20 mm to (175.6, 138.8)
- moved J5 0.20 mm to (162.4, 138.8)
Routing:
- net GND: track 169.7 -> 170.3 mm, vias 189 -> 193
- net (no net): vias 1 -> 0
Other:
- board size 35.1 x 50.4 mm -> 35.1 x 49.8 mm
- board text added: "ESP32 Breakout Board SMD rev 0.2 2019.07.08 rabbit-note.com"
- board text removed: "ESP32 Breakout Board SMD rev 0.1 2019.06.15 rabbit-note.com"
