File: ESP32-breakout-THD.kicad_pcb (KiCad board)
At the start: 2 copper layers, 35.1 x 50.4 mm, 16 parts, among them J1 Conn_01x14, J2 Conn_01x14, J3 Conn_01x02_Male, J4 Conn_01x04_Male, J5 Conn_01x04_Male, SW1 RESET, SW2 BOOT, U1 ESP32-WROOM

Commit message: fix: 微修正
Parts:
- removed the REF** at (160.5, 128.9)
- removed the REF** at (163.1, 128.9)
- added REF**: PinHeader_1x01_P2.54mm_Vertical, Connector_PinHeader_2.54mm:PinHeader_1x01_P2.54mm_Vertical, F.Cu at (163.1, 128.9)
- added REF**: PinHeader_1x01_P2.54mm_Vertical, Connector_PinHeader_2.54mm:PinHeader_1x01_P2.54mm_Vertical, F.Cu at (160.5, 128.9)
- C1, C2, C4: footprint Capacitor_SMD:C_0805_2012Metric -> Capacitor_SMD:C_0805_2012Metric_Pad1.15x1.40mm_HandSolder
- R1: footprint Resistor_SMD:R_0805_2012Metric -> Resistor_SMD:R_0805_2012Metric_Pad1.15x1.40mm_HandSolder
- REF**: value PinHeader_1x01_P1.27mm_Vertical -> PinHeader_1x01_P2.54mm_Vertical; footprint Connector_PinHeader_1.27mm:PinHeader_1x01_P1.27mm_Vertical -> Connector_PinHeader_2.54mm:PinHeader_1x01_P2.54mm_Vertical
- moved C4 0.48 mm to (164.1, 122.0)
Routing:
- net Net-(J1-Pad10): track 65.9 -> 67.4 mm
- net Net-(C4-Pad1): track 46.0 -> 46.6 mm
Other:
- board text added: "ESP32 Breakout Board rev 0.4 2019.07.08 rabbit-note.com"
- board text removed: "ESP32 Breakout Board rev 0.3 2019.06.14 rabbit-note.com"
