File: ESP32-breakout-THD.sch (KiCad schematic (older format))
At the start: 13 parts, among them J1 Conn_01x14, J2 Conn_01x14, J3 Conn_01x02_Male, J4 Conn_01x04_Male, J5 Conn_01x04_Male, SW1 RESET, SW2 BOOT, U1 ESP32-WROOM

Commit message: fix: 微修正
Parts:
- C1, C2, C4: footprint Capacitor_SMD:C_0805_2012Metric -> Capacitor_SMD:C_0805_2012Metric_Pad1.15x1.40mm_HandSolder
- C3: footprint Capacitor_SMD:C_1206_3216Metric -> Capacitor_SMD:C_1206_3216Metric_Pad1.42x1.75mm_HandSolder
- R1: footprint Resistor_SMD:R_0805_2012Metric -> Resistor_SMD:R_0805_2012Metric_Pad1.15x1.40mm_HandSolder
Changed lines of the file:
@@
 EESchema Schematic File Version 4
-LIBS:ESP32-breakout-cache
+LIBS:ESP32-breakout-THD-cache
 EELAYER 29 0
 EELAYER END
@@
 F 0 "R1" H 3320 2596 50  0000 L CNN
 F 1 "10k" H 3320 2505 50  0000 L CNN
-F 2 "Resistor_SMD:R_0805_2012Metric" V 3180 2550 50  0001 C CNN
+F 2 "Resistor_SMD:R_0805_2012Metric_Pad1.15x1.40mm_HandSolder" V 3180 2550 50  0001 C CNN
 F 3 "~" H 3250 2550 50  0001 C CNN
 	1    3250 2550
@@
 F 0 "C4" H 2765 4596 50  0000 L CNN
 F 1 "0.1u" H 2765 4505 50  0000 L CNN
-F 2 "Capacitor_SMD:C_0805_2012Metric" H 2688 4400 50  0001 C CNN
+F 2 "Capacitor_SMD:C_0805_2012Metric_Pad1.15x1.40mm_HandSolder" H 2688 4400 50  0001 C CNN
 F 3 "~" H 2650 4550 50  0001 C CNN
 	1    2650 4550
@@
 F 0 "C2" H 4565 4596 50  0000 L CNN
 F 1 "0.1u" H 4565 4505 50  0000 L CNN
-F 2 "Capacitor_SMD:C_0805_2012Metric" H 4488 4400 50  0001 C CNN
+F 2 "Capacitor_SMD:C_0805_2012Metric_Pad1.15x1.40mm_HandSolder" H 4488 4400 50  0001 C CNN
 F 3 "~" H 4450 4550 50  0001 C CNN
 	1    4450 4550
@@
 F 0 "C1" H 4165 4596 50  0000 L CNN
 F 1 "10u" H 4165 4505 50  0000 L CNN
-F 2 "Capacitor_SMD:C_0805_2012Metric" H 4088 4400 50  0001 C CNN
+F 2 "Capacitor_SMD:C_0805_2012Metric_Pad1.15x1.40mm_HandSolder" H 4088 4400 50  0001 C CNN
 F 3 "~" H 4050 4550 50  0001 C CNN
 	1    4050 4550
@@
 F 0 "C3" H 3765 4596 50  0000 L CNN
 F 1 "47u" H 3765 4505 50  0000 L CNN
-F 2 "Capacitor_SMD:C_1206_3216Metric" H 3688 4400 50  0001 C CNN
+F 2 "Capacitor_SMD:C_1206_3216Metric_Pad1.42x1.75mm_HandSolder" H 3688 4400 50  0001 C CNN
 F 3 "~" H 3650 4550 50  0001 C CNN
 	1    3650 4550
